File: pcb/mobo/mobo.kicad_sch (KiCad schematic)
At the start: 72 parts, among them J1 SWD_10, J2 PEEL_MOTOR, J3 DRIVE_MOTOR, J5 SPRING_FINGERS, J8 USART1, J9 SWD_10, U1 STM32F031C6Tx, U2 STM32F031K6Ux, U4 AP1117-33, U5 MC34063AD, U6 MAX3078E, U7 DRV8837, U8 DRV8837, Y1 8MHz

Commit message: updated to 8mm filter cap footprint
Parts:
- C16: footprint Capacitor_SMD:C_Elec_6.3x7.7 -> Capacitor_SMD:C_Elec_8x10.2
Changed lines of the file:
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@@
       (effects (font (size 1.27 1.27)) (justify left))
     )
-    (property "Footprint" "Capacitor_SMD:C_Elec_6.3x7.7" (at 88.9 224.79 0)
+    (property "Footprint" "Capacitor_SMD:C_Elec_8x10.2" (at 88.9 224.79 0)
       (effects (font (size 1.27 1.27)) hide)
     )
